Commit message: not fully functional but walkable

File: resources/robots/hr_URDF_1023/meshes/hr_URDF_1023.urdf (robot description, URDF)
Before this commit: robot hr_URDF_1023, 14 links, 13 joints
Links:
- link anklel: geometry collision mesh filename=../meshes/anklel.STL; visual mesh filename=../meshes/anklel.STL
- link ankler: geometry collision mesh filename=../meshes/ankler.STL; visual mesh filename=../meshes/ankler.STL
- link body: geometry collision box size=0.4 0.4 0.4; visual mesh filename=../meshes/body.STL
- link feetl: geometry collision mesh filename=../meshes/feetl.STL; visual mesh filename=../meshes/feetl.STL
- link feetr: geometry collision mesh filename=../meshes/feetr.STL; visual mesh filename=../meshes/feetr.STL
- link hip1l: geometry collision mesh filename=../meshes/hip1l.STL; visual mesh filename=../meshes/hip1l.STL
- link hip1r: geometry collision mesh filename=../meshes/hip1r.STL; visual mesh filename=../meshes/hip1r.STL
- link hip2l: geometry collision mesh filename=../meshes/hip2l.STL; visual mesh filename=../meshes/hip2l.STL
- link hip2r: geometry collision mesh filename=../meshes/hip2r.STL; visual mesh filename=../meshes/hip2r.STL
- link hip3l: geometry collision mesh filename=../meshes/hip3l.STL; visual mesh filename=../meshes/hip3l.STL
- link hip3r: geometry collision mesh filename=../meshes/hip3r.STL; visual mesh filename=../meshes/hip3r.STL
- link kneel: geometry collision mesh filename=../meshes/kneel.STL; visual mesh filename=../meshes/kneel.STL
- link kneer: geometry collision mesh filename=../meshes/kneer.STL; visual mesh filename=../meshes/kneer.STL
- link waist: geometry collision mesh filename=../meshes/waist.STL; visual mesh filename=../meshes/waist.STL
Joints:
- removed joint knee_yaw_l
- removed joint knee_yaw_r
- added joint hip_yaw_l: type revolute, parent hip2l, child hip3l, origin xyz=0 0 -0.17 rpy=0 0 0, axis 0 0 1, limit lower=-0.69813 upper=0.69813 effort=250 velocity=10
- added joint hip_yaw_r: type revolute, parent hip2r, child hip3r, origin xyz=0 0 -0.17 rpy=0 0 0, axis 0 0 1, limit lower=-0.69813 upper=0.69813 effort=250 velocity=10
- joint ankle_pitch_l: limit lower=-0.43644 upper=1.21087 effort=0 velocity=0 -> lower=-0.43644 upper=1.21087 effort=100 velocity=12
- joint ankle_pitch_r: limit lower=-0.43644 upper=1.21087 effort=0 velocity=0 -> lower=-0.43644 upper=1.21087 effort=100 velocity=12
- joint ankle_roll_l: limit lower=-0.43633 upper=0.43633 effort=0 velocity=0 -> lower=-0.43633 upper=0.43633 effort=100 velocity=12
- joint ankle_roll_r: limit lower=-0.43633 upper=0.43633 effort=0 velocity=0 -> lower=-0.43633 upper=0.43633 effort=100 velocity=12
- joint hip_pitch_l: limit lower=-0.7854 upper=1.8326 effort=0 velocity=0 -> lower=-0.7854 upper=1.7 effort=250 velocity=10
- joint hip_pitch_r: limit lower=-0.7854 upper=1.8326 effort=0 velocity=0 -> lower=-0.7854 upper=1.7 effort=250 velocity=10
- joint hip_roll_l: limit lower=-0.17453 upper=0.43633 effort=0 velocity=0 -> lower=-0.17453 upper=0.43633 effort=250 velocity=10
- joint hip_roll_r: limit lower=-0.43633 upper=0.17453 effort=0 velocity=0 -> lower=-0.43633 upper=0.17453 effort=250 velocity=10
- joint hip_yaw: limit lower=-3.14 upper=3.14 effort=0 velocity=0 -> lower=-3.14 upper=3.14 effort=250 velocity=12; type revolute -> fixed
- joint knee_pitch_l: limit lower=-2.36 upper=0 effort=0 velocity=0 -> lower=-2 upper=0 effort=250 velocity=12
- joint knee_pitch_r: limit lower=-2.36 upper=0 effort=0 velocity=0 -> lower=-2 upper=0 effort=250 velocity=10

File: resources/robots/hr_URDF_1023/urdf/hr_URDF_1023.urdf (robot description, URDF)
Before this commit: robot hr_URDF_1023, 14 links, 13 joints
Links:
- link anklel: geometry visual mesh filename=../meshes/anklel.STL
- link ankler: geometry visual mesh filename=../meshes/ankler.STL
- link body: geometry collision box size=0.4 0.4 0.4; visual mesh filename=../meshes/body.STL
- link hip1l: geometry visual mesh filename=../meshes/hip1l.STL
- link hip1r: geometry visual mesh filename=../meshes/hip1r.STL
- link hip2l: geometry visual mesh filename=../meshes/hip2l.STL
- link hip2r: geometry visual mesh filename=../meshes/hip2r.STL
- link hip3l: geometry visual mesh filename=../meshes/hip3l.STL
- link hip3r: geometry visual mesh filename=../meshes/hip3r.STL
- link kneel: geometry visual mesh filename=../meshes/kneel.STL
- link kneer: geometry visual mesh filename=../meshes/kneer.STL
- link waist: geometry visual mesh filename=../meshes/waist.STL
Joints:
- removed joint knee_yaw_l
- removed joint knee_yaw_r
- added joint hip_yaw_l: type revolute, parent hip2l, child hip3l, origin xyz=0 0 -0.17 rpy=0 0 0, axis 0 0 1, limit lower=-0.69813 upper=0.69813 effort=1000 velocity=1000
- added joint hip_yaw_r: type revolute, parent hip2r, child hip3r, origin xyz=0 0 -0.17 rpy=0 0 0, axis 0 0 1, limit lower=-0.69813 upper=0.69813 effort=1000 velocity=1000
- joint ankle_pitch_l: limit lower=-0.43644 upper=1.21087 effort=0 velocity=0 -> lower=-0.43644 upper=1.21087 effort=700 velocity=400
- joint ankle_pitch_r: limit lower=-0.43644 upper=1.21087 effort=0 velocity=0 -> lower=-0.43644 upper=1.21087 effort=700 velocity=400
- joint ankle_roll_l: limit lower=-0.43633 upper=0.43633 effort=0 velocity=0 -> lower=-0.43633 upper=0.43633 effort=700 velocity=400
- joint ankle_roll_r: limit lower=-0.43633 upper=0.43633 effort=0 velocity=0 -> lower=-0.43633 upper=0.43633 effort=700 velocity=400
- joint hip_pitch_l: limit lower=-0.7854 upper=1.8326 effort=0 velocity=0 -> lower=-0.7854 upper=1.7 effort=1000 velocity=1000
- joint hip_pitch_r: limit lower=-0.7854 upper=1.8326 effort=0 velocity=0 -> lower=-0.7854 upper=1.7 effort=1000 velocity=1000
- joint hip_roll_l: limit lower=-0.17453 upper=0.43633 effort=0 velocity=0 -> lower=-0.17453 upper=0.43633 effort=1000 velocity=1000
- joint hip_roll_r: limit lower=-0.43633 upper=0.17453 effort=0 velocity=0 -> lower=-0.43633 upper=0.17453 effort=1000 velocity=1000
- joint hip_yaw: limit lower=-3.14 upper=3.14 effort=0 velocity=0 -> lower=-3.14 upper=3.14 effort=1000 velocity=1000; type revolute -> fixed
- joint knee_pitch_l: limit lower=-2.36 upper=0 effort=0 velocity=0 -> lower=-2 upper=0 effort=1000 velocity=1000
- joint knee_pitch_r: limit lower=-2.36 upper=0 effort=0 velocity=0 -> lower=-2 upper=0 effort=1000 velocity=1000

Commit message: 20250407

File: resources/robots/hr_URDF_1023/meshes/hr_URDF_1023.urdf (robot description, URDF)
Before this commit: robot hr_URDF_1023, 14 links, 13 joints
Links:
- link anklel: geometry visual mesh filename=../meshes/anklel.STL
- link ankler: geometry visual mesh filename=../meshes/ankler.STL
- link body: mass 20.6588 -> 10.6588
- link hip1l: geometry visual mesh filename=../meshes/hip1l.STL
- link hip1r: geometry visual mesh filename=../meshes/hip1r.STL
- link hip2l: geometry visual mesh filename=../meshes/hip2l.STL
- link hip2r: geometry visual mesh filename=../meshes/hip2r.STL
- link hip3l: geometry visual mesh filename=../meshes/hip3l.STL
- link hip3r: geometry visual mesh filename=../meshes/hip3r.STL
- link kneel: geometry visual mesh filename=../meshes/kneel.STL
- link kneer: geometry visual mesh filename=../meshes/kneer.STL
- link waist: geometry visual mesh filename=../meshes/waist.STL
Joints:
- joint ankle_pitch_l: limit lower=-0.43644 upper=1.21087 effort=100 velocity=12 -> lower=-0.43644 upper=1.21087 effort=700 velocity=400
- joint ankle_pitch_r: limit lower=-0.43644 upper=1.21087 effort=100 velocity=12 -> lower=-0.43644 upper=1.21087 effort=700 velocity=400
- joint ankle_roll_l: limit lower=-0.43633 upper=0.43633 effort=100 velocity=12 -> lower=-0.43633 upper=0.43633 effort=700 velocity=400
- joint ankle_roll_r: limit lower=-0.43633 upper=0.43633 effort=100 velocity=12 -> lower=-0.43633 upper=0.43633 effort=700 velocity=400
- joint hip_pitch_l: limit lower=-0.7854 upper=1.7 effort=250 velocity=10 -> lower=-0.7854 upper=1.7 effort=1000 velocity=1000
- joint hip_pitch_r: limit lower=-0.7854 upper=1.7 effort=250 velocity=10 -> lower=-0.7854 upper=1.7 effort=1000 velocity=1000
- joint hip_roll_l: limit lower=-0.17453 upper=0.43633 effort=250 velocity=10 -> lower=-0.17453 upper=0.43633 effort=1000 velocity=1000
- joint hip_roll_r: limit lower=-0.43633 upper=0.17453 effort=250 velocity=10 -> lower=-0.43633 upper=0.17453 effort=1000 velocity=1000
- joint hip_yaw: limit lower=-3.14 upper=3.14 effort=250 velocity=12 -> lower=-3.14 upper=3.14 effort=1000 velocity=1000
- joint hip_yaw_l: limit lower=-0.69813 upper=0.69813 effort=250 velocity=10 -> lower=-0.69813 upper=0.69813 effort=1000 velocity=1000
- joint hip_yaw_r: limit lower=-0.69813 upper=0.69813 effort=250 velocity=10 -> lower=-0.69813 upper=0.69813 effort=1000 velocity=1000
- joint knee_pitch_l: limit lower=-2 upper=0 effort=250 velocity=12 -> lower=-2 upper=0 effort=1000 velocity=1000
- joint knee_pitch_r: limit lower=-2 upper=0 effort=250 velocity=10 -> lower=-2 upper=0 effort=1000 velocity=1000

File: resources/robots/hr_URDF_1023/urdf/hr_URDF_1023.urdf (robot description, URDF)
Before this commit: robot hr_URDF_1023, 14 links, 13 joints
Links:
- link body: mass 20.6588 -> 10.6588
Joints:
- joint ankle_pitch_l: limit lower=-0.43644 upper=1.21087 effort=700 velocity=400 -> lower=-0.43644 upper=1.21087 effort=9999999 velocity=9999999
- joint ankle_pitch_r: limit lower=-0.43644 upper=1.21087 effort=700 velocity=400 -> lower=-0.43644 upper=1.21087 effort=9999999 velocity=9999999
- joint ankle_roll_l: limit lower=-0.43633 upper=0.43633 effort=700 velocity=400 -> lower=-0.43633 upper=0.43633 effort=9999999 velocity=9999999
- joint ankle_roll_r: limit lower=-0.43633 upper=0.43633 effort=700 velocity=400 -> lower=-0.43633 upper=0.43633 effort=9999999 velocity=9999999
- joint hip_pitch_l: limit lower=-0.7854 upper=1.7 effort=1000 velocity=1000 -> lower=-0.7854 upper=1.7 effort=9999999 velocity=9999999
- joint hip_pitch_r: limit lower=-0.7854 upper=1.7 effort=1000 velocity=1000 -> lower=-0.7854 upper=1.7 effort=9999999 velocity=9999999
- joint hip_roll_l: limit lower=-0.17453 upper=0.43633 effort=1000 velocity=1000 -> lower=-0.17453 upper=0.43633 effort=9999999 velocity=9999999
- joint hip_roll_r: limit lower=-0.43633 upper=0.17453 effort=1000 velocity=1000 -> lower=-0.43633 upper=0.17453 effort=9999999 velocity=9999999
- joint hip_yaw: limit lower=-3.14 upper=3.14 effort=1000 velocity=1000 -> lower=-3.14 upper=3.14 effort=9999999 velocity=9999999
- joint hip_yaw_l: limit lower=-0.69813 upper=0.69813 effort=1000 velocity=1000 -> lower=-0.69813 upper=0.69813 effort=9999999 velocity=9999999
- joint hip_yaw_r: limit lower=-0.69813 upper=0.69813 effort=1000 velocity=1000 -> lower=-0.69813 upper=0.69813 effort=9999999 velocity=9999999
- joint knee_pitch_l: limit lower=-2 upper=0 effort=1000 velocity=1000 -> lower=-2 upper=0 effort=9999999 velocity=9999999
- joint knee_pitch_r: limit lower=-2 upper=0 effort=1000 velocity=1000 -> lower=-2 upper=0 effort=9999999 velocity=9999999

Commit message: 20240410

File: resources/robots/hr_URDF_1023/meshes/hr_URDF_1023.urdf (robot description, URDF)
Before this commit: robot hr_URDF_1023, 14 links, 13 joints
Links:
- link body: mass 10.6588 -> 2.6588
Joints:
- joint ankle_pitch_l: limit lower=-0.43644 upper=1.21087 effort=700 velocity=400 -> lower=-0.43644 upper=1.21087 effort=9999999 velocity=9999999
- joint ankle_pitch_r: limit lower=-0.43644 upper=1.21087 effort=700 velocity=400 -> lower=-0.43644 upper=1.21087 effort=9999999 velocity=9999999
- joint ankle_roll_l: limit lower=-0.43633 upper=0.43633 effort=700 velocity=400 -> lower=-0.43633 upper=0.43633 effort=9999999 velocity=9999999
- joint ankle_roll_r: limit lower=-0.43633 upper=0.43633 effort=700 velocity=400 -> lower=-0.43633 upper=0.43633 effort=9999999 velocity=9999999
- joint hip_pitch_l: limit lower=-0.7854 upper=1.7 effort=1000 velocity=1000 -> lower=-0.7854 upper=1.7 effort=9999999 velocity=9999999
- joint hip_pitch_r: limit lower=-0.7854 upper=1.7 effort=1000 velocity=1000 -> lower=-0.7854 upper=1.7 effort=9999999 velocity=9999999
- joint hip_roll_l: limit lower=-0.17453 upper=0.43633 effort=1000 velocity=1000 -> lower=-0.17453 upper=0.43633 effort=9999999 velocity=9999999
- joint hip_roll_r: limit lower=-0.43633 upper=0.17453 effort=1000 velocity=1000 -> lower=-0.43633 upper=0.17453 effort=9999999 velocity=9999999
- joint hip_yaw: limit lower=-3.14 upper=3.14 effort=1000 velocity=1000 -> lower=-3.14 upper=3.14 effort=9999999 velocity=9999999
- joint hip_yaw_l: limit lower=-0.69813 upper=0.69813 effort=1000 velocity=1000 -> lower=-0.69813 upper=0.69813 effort=9999999 velocity=9999999
- joint hip_yaw_r: limit lower=-0.69813 upper=0.69813 effort=1000 velocity=1000 -> lower=-0.69813 upper=0.69813 effort=9999999 velocity=9999999
- joint knee_pitch_l: limit lower=-2 upper=0 effort=1000 velocity=1000 -> lower=-2 upper=0 effort=9999999 velocity=9999999
- joint knee_pitch_r: limit lower=-2 upper=0 effort=1000 velocity=1000 -> lower=-2 upper=0 effort=9999999 velocity=9999999
